File: documents/electronic design/UsbDevice/UsbDevice.sch (KiCad schematic (older format))
At the start: 3 parts

Commit message: update schematics and pcb projects
Parts:
- removed U? (x2): NRF24L01-BRKOUT, NRF24L01-BKKOUT, symbol NRF24L01-BRKOUT
- removed U?: STM32F103C8T6, LQFP48_7X7MM_0.5MMPP, symbol STM32F103C8T6
- added P1, P2: CONN_01X20, Pin_Headers:Pin_Header_Straight_1x20, symbol CONN_01X20
- added P?: CONN_STM32F103_L_01X20, symbol CONN_STM32F103_L_01X20
- added P?: CONN_STM32F103_R_01X20, symbol CONN_STM32F103_R_01X20-RESCUE-UsbDevice
- added U1, U2: NRF24L01-BRKOUT, se8r01_smd:SE8R01_SMD, symbol NRF24L01-BRKOUT-RESCUE-UsbDevice
Connections:
- net labels added: CE1, CE2, CSN_1, CSN_2, IRQ1, IRQ2, SPI1_MISO, SPI1_MOSI, SPI1_SCK
- net labels removed: MOSI
- wire segments 0 -> 31
- no-connect marks 0 -> 69
