File: documents/electronic design/beamer/_saved_beamer.sch (KiCad schematic (older format))
At the start: 23 parts, among them P1 CONN_01X20, P2 CONN_01X20, T1 2N7002K, T10 2N7002K, T2 2N7002K, T3 2N7002K, T4 2N7002K, T5 2N7002K, T6 2N7002K, T7 2N7002K, T8 2N7002K, T9 2N7002K, U1 NRF24L01-BRKOUT

Commit message: update schematics and pcb projects
Parts:
- T1, T10, T2, T3, T4, T5, T6, T7, T8, T9: footprint SOT23 -> 2N7002K:SOT23
- U1: footprint NRF24L01-BKKOUT -> se8r01_smd:SE8R01_SMD
Connections:
- net IR_PIN_1: now also P1.8 (P8); no longer P2.8 (P8)
- net IR_PIN_2: now also P1.9 (P9); no longer P2.7 (P7)
- net IR_PIN_3: now also P1.10 (P10); no longer P1.11 (P11)
- net IR_PIN_4: now also P1.11 (P11); no longer P1.12 (P12)
- net IR_PIN_5: now also P1.12 (P12); no longer P1.13 (P13)
- net IR_PIN_6: now also P1.13 (P13); no longer P1.14 (P14)
- net IR_PIN_7: now also P1.14 (P14); no longer P1.15 (P15)
- net IR_PIN_8: now also P1.15 (P15); no longer P1.16 (P16)
- net IR_PIN_ID: now also P1.16 (P16); no longer P1.1 (P1)
- no-connect marks 23 -> 22
Changed lines of the file:
@@
 EESchema Schematic File Version 2
+LIBS:power
+LIBS:device
+LIBS:transistors
+LIBS:conn
+LIBS:linear
+LIBS:regul
+LIBS:74xx
+LIBS:cmos4000
+LIBS:adc-dac
+LIBS:memory
+LIBS:xilinx
+LIBS:microcontrollers
+LIBS:dsp
+LIBS:microchip
+LIBS:analog_switches
+LIBS:motorola
+LIBS:texas
+LIBS:intel
+LIBS:audio
+LIBS:interface
+LIBS:digital-audio
+LIBS:philips
+LIBS:display
+LIBS:cypress
+LIBS:siliconi
+LIBS:opto
+LIBS:atmel
+LIBS:contrib
+LIBS:valves
+LIBS:2N7002K
 LIBS:NRF24L01-BRKOUT
-LIBS:ir_beamer-cache
+LIBS:conn_R
+LIBS:beamer-cache
 EELAYER 25 0
 EELAYER END
@@
 F 0 "T1" H 1150 2150 50  0000 L CNN
 F 1 "2N7002K" H 1000 2050 50  0000 L CNN
-F 2 "SOT23" H 1350 1900 50  0001 L CNN
+F 2 "2N7002K:SOT23" H 1350 1900 50  0001 L CNN
 F 3 "" H 1350 1900 60  0000 C CNN
 	1    1350 1900
@@
 F 0 "T4" H 2650 3050 50  0000 L CNN
 F 1 "2N7002K" H 2500 2950 50  0000 L CNN
-F 2 "SOT23" H 2850 2800 50  0001 L CNN
+F 2 "2N7002K:SOT23" H 2850 2800 50  0001 L CNN
 F 3 "" H 2850 2800 60  0000 C CNN
 	1    2850 2800
@@
 F 0 "T2" H 1750 2150 50  0000 L CNN
 F 1 "2N7002K" H 1600 2050 50  0000 L CNN
-F 2 "SOT23" H 1950 1900 50  0001 L CNN
+F 2 "2N7002K:SOT23" H 1950 1900 50  0001 L CNN
 F 3 "" H 1950 1900 60  0000 C CNN
 	1    1950 1900
@@
 F 0 "T3" H 2350 2150 50  0000 L CNN
 F 1 "2N7002K" H 2200 2050 50  0000 L CNN
-F 2 "SOT23" H 2550 1900 50  0001 L CNN
+F 2 "2N7002K:SOT23" H 2550 1900 50  0001 L CNN
 F 3 "" H 2550 1900 60  0000 C CNN
 	1    2550 1900
@@
 F 0 "T5" H 2950 2150 50  0000 L CNN
 F 1 "2N7002K" H 2800 2050 50  0000 L CNN
-F 2 "SOT23" H 3150 1900 50  0001 L CNN
+F 2 "2N7002K:SOT23" H 3150 1900 50  0001 L CNN
 F 3 "" H 3150 1900 60  0000 C CNN
 	1    3150 1900
@@
 F 0 "T6" H 3550 2150 50  0000 L CNN
 F 1 "2N7002K" H 3400 2050 50  0000 L CNN
-F 2 "SOT23" H 3750 1900 50  0001 L CNN
+F 2 "2N7002K:SOT23" H 3750 1900 50  0001 L CNN
 F 3 "" H 3750 1900 60  0000 C CNN
 	1    3750 1900
@@
 F 0 "T7" H 4150 2150 50  0000 L CNN
 F 1 "2N7002K" H 4000 2050 50  0000 L CNN
-F 2 "SOT23" H 4350 1900 50  0001 L CNN
+F 2 "2N7002K:SOT23" H 4350 1900 50  0001 L CNN
 F 3 "" H 4350 1900 60  0000 C CNN
 	1    4350 1900
@@
 F 0 "T8" H 4750 2150 50  0000 L CNN
 F 1 "2N7002K" H 4600 2050 50  0000 L CNN
-F 2 "SOT23" H 4950 1900 50  0001 L CNN
+F 2 "2N7002K:SOT23" H 4950 1900 50  0001 L CNN
 F 3 "" H 4950 1900 60  0000 C CNN
 	1    4950 1900
@@
 F 0 "T9" H 5350 2150 50  0000 L CNN
 F 1 "2N7002K" H 5200 2050 50  0000 L CNN
-F 2 "SOT23" H 5550 1900 50  0001 L CNN
+F 2 "2N7002K:SOT23" H 5550 1900 50  0001 L CNN
 F 3 "" H 5550 1900 60  0000 C CNN
 	1    5550 1900
@@
 F 0 "T10" H 6600 2150 50  0000 L CNN
 F 1 "2N7002K" H 6450 2050 50  0000 L CNN
-F 2 "SOT23" H 6800 1900 50  0001 L CNN
+F 2 "2N7002K:SOT23" H 6800 1900 50  0001 L CNN
 F 3 "" H 6800 1900 60  0000 C CNN
 	1    6800 1900
@@
 Text GLabel 4450 5300 0    60   Input ~ 0
 NRF_IRQ1
-Text GLabel 4450 4300 0    60   Input ~ 0
+Text GLabel 2900 4300 2    60   Input ~ 0
 IR_PIN_1
-Text GLabel 4450 4200 0    60   Input ~ 0
+Text GLabel 2900 4400 2    60   Input ~ 0
 IR_PIN_2
+Text GLabel 2900 4500 2    60   Input ~ 0
+IR_PIN_3
 Text GLabel 2900 4600 2    60   Input ~ 0
-IR_PIN_3
+IR_PIN_4
 Text GLabel 2900 4700 2    60   Input ~ 0
-IR_PIN_4
+IR_PIN_5
 Text GLabel 2900 4800 2    60   Input ~ 0
-IR_PIN_5
+IR_PIN_6
 Text GLabel 2900 4900 2    60   Input ~ 0
-IR_PIN_6
+IR_PIN_7
 Text GLabel 2900 5000 2    60   Input ~ 0
-IR_PIN_7
+IR_PIN_8
 Text GLabel 2900 5100 2    60   Input ~ 0
-IR_PIN_8
-Text GLabel 2900 3600 2    60   Input ~ 0
 IR_PIN_ID
 NoConn ~ 2800 5500
 NoConn ~ 2800 5400
 NoConn ~ 2800 5300
-NoConn ~ 2800 4500
-NoConn ~ 2800 4400
-NoConn ~ 2800 4300
 NoConn ~ 2800 4200
 NoConn ~ 2800 4100
@@
 Text GLabel 2900 5200 2    60   Input ~ 0
 PWM_38K
-NoConn ~ 4500 3650
 $Comp
 L GND #PWR05
@@
 	2800 5200 2900 5200
 Wire Wire Line
-	2800 3600 2900 3600
-Wire Wire Line
 	4050 3450 4500 3450
 Wire Wire Line
@@
 Wire Wire Line
 	8400 1750 8600 1750
+Wire Wire Line
+	2800 4400 2900 4400
+Wire Wire Line
+	2800 4500 2900 4500
+NoConn ~ 4450 4300
+NoConn ~ 4450 4200
+Wire Wire Line
+	2800 4300 2900 4300
+NoConn ~ 2800 3600
 $Comp
 L NRF24L01-BRKOUT U1
-U 1 1 5713BCFC
+U 1 1 571409CC
 P 9200 1850
 F 0 "U1" H 8800 2450 50  0000 L CNN
 F 1 "NRF24L01-BRKOUT" H 9200 1250 50  0000 L CNN
-F 2 "NRF24L01-BKKOUT" H 9200 1850 50  0001 L CNN
+F 2 "se8r01_smd:SE8R01_SMD" H 9200 1850 50  0001 L CNN
 F 3 "" H 9200 1850 60  0000 C CNN
 	1    9200 1850
