File: documents/electronic design/beamer/_saved_beamer.sch (KiCad schematic (older format))
At the start: 23 parts, among them P1 CONN_01X20, P2 CONN_01X20, T1 2N7002K, T10 2N7002K, T2 2N7002K, T3 2N7002K, T4 2N7002K, T5 2N7002K, T6 2N7002K, T7 2N7002K, T8 2N7002K, T9 2N7002K, U1 NRF24L01-BRKOUT

Commit message: add capacitor to pcb
Parts:
- added C1: C, Capacitors_SMD:C_1210_HandSoldering, symbol C
- U1: footprint se8r01_smd:SE8R01_SMD -> NRF24L01-BKKOUT
Connections:
- net +3V3: now also C1.2
- net GND: now also C1.1
Changed lines of the file:
@@
 L GND #PWR05
 U 1 1 57142C4E
-P 8400 1550
-F 0 "#PWR05" H 8400 1300 50  0001 C CNN
-F 1 "GND" H 8400 1400 50  0000 C CNN
-F 2 "" H 8400 1550 50  0000 C CNN
-F 3 "" H 8400 1550 50  0000 C CNN
-	1    8400 1550
+P 8350 1500
+F 0 "#PWR05" H 8350 1250 50  0001 C CNN
+F 1 "GND" H 8350 1350 50  0000 C CNN
+F 2 "" H 8350 1500 50  0000 C CNN
+F 3 "" H 8350 1500 50  0000 C CNN
+	1    8350 1500
 	0    1    1    0
 $EndComp
@@
 L +3.3V #PWR06
 U 1 1 57142CA4
-P 8400 1750
-F 0 "#PWR06" H 8400 1600 50  0001 C CNN
-F 1 "+3.3V" H 8400 1890 50  0000 C CNN
-F 2 "" H 8400 1750 50  0000 C CNN
-F 3 "" H 8400 1750 50  0000 C CNN
-	1    8400 1750
+P 8350 1800
+F 0 "#PWR06" H 8350 1650 50  0001 C CNN
+F 1 "+3.3V" H 8350 1940 50  0000 C CNN
+F 2 "" H 8350 1800 50  0000 C CNN
+F 3 "" H 8350 1800 50  0000 C CNN
+	1    8350 1800
 	0    -1   -1   0
 $EndComp
-$Comp
-L PWR_FLAG #FLG07
-U 1 1 57142E4E
-P 4050 3450
-F 0 "#FLG07" H 4050 3545 50  0001 C CNN
-F 1 "PWR_FLAG" H 4050 3630 50  0000 C CNN
-F 2 "" H 4050 3450 50  0000 C CNN
-F 3 "" H 4050 3450 50  0000 C CNN
-	1    4050 3450
-	1    0    0    -1
-$EndComp
-$Comp
-L PWR_FLAG #FLG08
-U 1 1 57142EAB
-P 4050 3850
-F 0 "#FLG08" H 4050 3945 50  0001 C CNN
-F 1 "PWR_FLAG" H 4050 4030 50  0000 C CNN
-F 2 "" H 4050 3850 50  0000 C CNN
-F 3 "" H 4050 3850 50  0000 C CNN
-	1    4050 3850
-	1    0    0    -1
-$EndComp
-Wire Wire Line
-	9800 1550 9900 1550
-Wire Wire Line
-	9800 1750 9900 1750
-Wire Wire Line
-	9800 1950 9900 1950
-Wire Wire Line
-	9800 2150 9900 2150
-Wire Wire Line
-	8600 2150 8500 2150
-Wire Wire Line
-	8600 1950 8500 1950
-Wire Wire Line
-	1450 1600 1450 1500
-Wire Wire Line
-	2950 800  2950 750
-Wire Wire Line
-	2050 1600 2050 1500
-Wire Wire Line
-	2650 1600 2650 1500
-Wire Wire Line
-	3250 1600 3250 1500
-Wire Wire Line
-	3850 1600 3850 1500
-Wire Wire Line
-	4450 1600 4450 1500
-Wire Wire Line
-	5050 1600 5050 1500
-Wire Wire Line
-	5650 1600 5650 1500
-Wire Wire Line
-	1450 1100 6900 1100
-Connection ~ 2650 1100
-Connection ~ 2050 1100
-Connection ~ 2950 1100
-Connection ~ 3250 1100
-Connection ~ 3850 1100
-Connection ~ 4450 1100
-Connection ~ 5050 1100
-Wire Wire Line
-	1050 1900 1150 1900
-Wire Wire Line
-	1650 1900 1750 1900
-Wire Wire Line
-	2250 1900 2350 1900
-Wire Wire Line
-	2850 1900 2950 1900
-Wire Wire Line
-	3450 1900 3550 1900
-Wire Wire Line
-	4050 1900 4150 1900
-Wire Wire Line
-	4650 1900 4750 1900
-Wire Wire Line
-	5250 1900 5350 1900
-Wire Wire Line
-	6900 1600 6900 1500
-Wire Wire Line
-	6500 1900 6600 1900
-Connection ~ 5650 1100
-Wire Wire Line
-	2550 2800 2650 2800
-Wire Wire Line
-	2950 3100 2950 3000
-Wire Wire Line
-	2650 2100 2650 2500
-Wire Wire Line
-	1450 2500 6900 2500
-Wire Wire Line
-	2050 2100 2050 2500
-Connection ~ 2650 2500
-Wire Wire Line
-	1450 2100 1450 2500
-Connection ~ 2050 2500
-Wire Wire Line
-	3250 2100 3250 2500
-Connection ~ 2950 2500
-Wire Wire Line
-	3850 2500 3850 2100
-Connection ~ 3250 2500
-Wire Wire Line
-	4450 2500 4450 2100
-Connection ~ 3850 2500
-Wire Wire Line
-	5050 2500 5050 2100
-Connection ~ 4450 2500
-Wire Wire Line
-	5650 2500 5650 2100
-Connection ~ 5050 2500
-Wire Wire Line
-	6900 2500 6900 2100
-Connection ~ 5650 2500
-Wire Wire Line
-	4450 4400 4550 4400
-Wire Wire Line
-	4450 4500 4550 4500
-Wire Wire Line
-	4450 4600 4550 4600
-Wire Wire Line
-	4450 5100 4550 5100
-Wire Wire Line
-	4450 5200 4550 5200
-Wire Wire Line
-	4450 5300 4550 5300
-Wire Wire Line
-	2800 4600 2900 4600
-Wire Wire Line
-	2800 4700 2900 4700
-Wire Wire Line
-	2800 4800 2900 4800
-Wire Wire Line
-	2800 4900 2900 4900
-Wire Wire Line
-	2800 5000 2900 5000
-Wire Wire Line
-	2800 5100 2900 5100
-Wire Wire Line
-	4450 3800 4550 3800
-Wire Wire Line
-	4450 3600 4550 3600
-Wire Wire Line
-	2800 5200 2900 5200
-Wire Wire Line
-	4050 3450 4500 3450
-Wire Wire Line
-	4500 3450 4500 3700
-Connection ~ 4500 3600
-Wire Wire Line
-	4050 3850 4050 3950
-Wire Wire Line
-	4050 3950 4500 3950
-Wire Wire Line
-	4500 3950 4500 3800
-Connection ~ 4500 3800
-Wire Wire Line
-	8600 1550 8400 1550
-Wire Wire Line
-	8400 1750 8600 1750
-$Comp
-L NRF24L01-BRKOUT U1
-U 1 1 5713E8BE
-P 9200 1850
-F 0 "U1" H 8800 2450 50  0000 L CNN
-F 1 "NRF24L01-BRKOUT" H 9200 1250 50  0000 L CNN
-F 2 "se8r01_smd:SE8R01_SMD" H 9200 1850 50  0001 L CNN
-F 3 "" H 9200 1850 60  0000 C CNN
-	1    9200 1850
-	1    0    0    -1
-$EndComp
-Wire Wire Line
-	2800 4400 2900 4400
-Wire Wire Line
-	2800 4500 2900 4500
 NoConn ~ 4550 4300
 NoConn ~ 4550 4200
-Wire Wire Line
-	2800 4300 2900 4300
 NoConn ~ 2800 3600
 $Comp
-L +3.3V #PWR09
+L +3.3V #PWR07
 U 1 1 57153B7B
 P 2900 5500
-F 0 "#PWR09" H 2900 5350 50  0001 C CNN
+F 0 "#PWR07" H 2900 5350 50  0001 C CNN
 F 1 "+3.3V" H 2900 5640 50  0000 C CNN
 F 2 "" H 2900 5500 50  0000 C CNN
@@
 $EndComp
 $Comp
-L GND #PWR010
+L GND #PWR08
 U 1 1 57153C2F
 P 2900 5400
-F 0 "#PWR010" H 2900 5150 50  0001 C CNN
+F 0 "#PWR08" H 2900 5150 50  0001 C CNN
 F 1 "GND" H 2900 5250 50  0000 C CNN
 F 2 "" H 2900 5400 50  0000 C CNN
@@
 	0    -1   -1   0
 $EndComp
+$Comp
+L C C1
+U 1 1 57177FF4
+P 8350 1650
+F 0 "C1" H 8375 1750 50  0000 L CNN
+F 1 "C" H 8375 1550 50  0000 L CNN
+F 2 "Capacitors_SMD:C_1210_HandSoldering" H 8388 1500 50  0001 C CNN
+F 3 "" H 8350 1650 50  0000 C CNN
+	1    8350 1650
+	1    0    0    -1
+$EndComp
+$Comp
+L PWR_FLAG #FLG09
+U 1 1 57142E4E
+P 4050 3450
+F 0 "#FLG09" H 4050 3545 50  0001 C CNN
+F 1 "PWR_FLAG" H 4050 3630 50  0000 C CNN
+F 2 "" H 4050 3450 50  0000 C CNN
+F 3 "" H 4050 3450 50  0000 C CNN
+	1    4050 3450
+	1    0    0    -1
+$EndComp
+$Comp
+L PWR_FLAG #FLG010
+U 1 1 57142EAB
+P 4050 3850
+F 0 "#FLG010" H 4050 3945 50  0001 C CNN
+F 1 "PWR_FLAG" H 4050 4030 50  0000 C CNN
+F 2 "" H 4050 3850 50  0000 C CNN
+F 3 "" H 4050 3850 50  0000 C CNN
+	1    4050 3850
+	1    0    0    -1
+$EndComp
+Wire Wire Line
+	4050 3450 4500 3450
+Wire Wire Line
+	4500 3450 4500 3700
+Wire Wire Line
+	4050 3950 4500 3950
+Wire Wire Line
+	4500 3950 4500 3800
+Wire Wire Line
+	4050 3850 4050 3950
+Wire Wire Line
+	8500 1800 8350 1800
+Wire Wire Line
+	8500 1750 8500 1800
+Wire Wire Line
+	8600 1750 8500 1750
+Wire Wire Line
+	8500 1500 8350 1500
+Wire Wire Line
+	8500 1550 8500 1500
+Wire Wire Line
+	8600 1550 8500 1550
+Wire Wire Line
+	4500 3700 4550 3700
+Wire Wire Line
+	2800 5400 2900 5400
 Wire Wire Line
 	2800 5500 2900 5500
 Wire Wire Line
-	2800 5400 2900 5400
-Wire Wire Line
-	4500 3700 4550 3700
+	2800 4300 2900 4300
+Wire Wire Line
+	2800 4500 2900 4500
+Wire Wire Line
+	2800 4400 2900 4400
+Connection ~ 4500 3800
+Connection ~ 4500 3600
+Wire Wire Line
+	2800 5200 2900 5200
+Wire Wire Line
+	4450 3600 4550 3600
+Wire Wire Line
+	4450 3800 4550 3800
+Wire Wire Line
+	2800 5100 2900 5100
+Wire Wire Line
+	2800 5000 2900 5000
+Wire Wire Line
+	2800 4900 2900 4900
+Wire Wire Line
+	2800 4800 2900 4800
+Wire Wire Line
+	2800 4700 2900 4700
+Wire Wire Line
+	2800 4600 2900 4600
+Wire Wire Line
+	4450 5300 4550 5300
+Wire Wire Line
+	4450 5200 4550 5200
+Wire Wire Line
+	4450 5100 4550 5100
+Wire Wire Line
+	4450 4600 4550 4600
+Wire Wire Line
+	4450 4500 4550 4500
+Wire Wire Line
+	4450 4400 4550 4400
+Connection ~ 5650 2500
+Wire Wire Line
+	6900 2500 6900 2100
+Connection ~ 5050 2500
+Wire Wire Line
+	5650 2500 5650 2100
+Connection ~ 4450 2500
+Wire Wire Line
+	5050 2500 5050 2100
+Connection ~ 3850 2500
+Wire Wire Line
+	4450 2500 4450 2100
+Connection ~ 3250 2500
+Wire Wire Line
+	3850 2500 3850 2100
+Connection ~ 2950 2500
+Wire Wire Line
+	3250 2100 3250 2500
+Connection ~ 2050 2500
+Wire Wire Line
+	1450 2100 1450 2500
+Connection ~ 2650 2500
+Wire Wire Line
+	2050 2100 2050 2500
+Wire Wire Line
+	1450 2500 6900 2500
+Wire Wire Line
+	2650 2100 2650 2500
+Wire Wire Line
+	2950 3100 2950 3000
+Wire Wire Line
+	2550 2800 2650 2800
+Connection ~ 5650 1100
+Wire Wire Line
+	6500 1900 6600 1900
+Wire Wire Line
+	6900 1600 6900 1500
+Wire Wire Line
+	5250 1900 5350 1900
+Wire Wire Line
+	4650 1900 4750 1900
+Wire Wire Line
+	4050 1900 4150 1900
+Wire Wire Line
+	3450 1900 3550 1900
+Wire Wire Line
+	2850 1900 2950 1900
+Wire Wire Line
+	2250 1900 2350 1900
+Wire Wire Line
+	1650 1900 1750 1900
+Wire Wire Line
+	1050 1900 1150 1900
+Connection ~ 5050 1100
+Connection ~ 4450 1100
+Connection ~ 3850 1100
+Connection ~ 3250 1100
+Connection ~ 2950 1100
+Connection ~ 2050 1100
+Connection ~ 2650 1100
+Wire Wire Line
+	1450 1100 6900 1100
+Wire Wire Line
+	5650 1600 5650 1500
+Wire Wire Line
+	5050 1600 5050 1500
+Wire Wire Line
+	4450 1600 4450 1500
+Wire Wire Line
+	3850 1600 3850 1500
+Wire Wire Line
+	3250 1600 3250 1500
+Wire Wire Line
+	2650 1600 2650 1500
+Wire Wire Line
+	2050 1600 2050 1500
+Wire Wire Line
+	2950 800  2950 750
+Wire Wire Line
+	1450 1600 1450 1500
+Wire Wire Line
+	8600 1950 8500 1950
+Wire Wire Line
+	8600 2150 8500 2150
+Wire Wire Line
+	9800 2150 9900 2150
+Wire Wire Line
+	9800 1950 9900 1950
+Wire Wire Line
+	9800 1750 9900 1750
+Wire Wire Line
+	9800 1550 9900 1550
+$Comp
+L NRF24L01-BRKOUT U1
+U 1 1 571793F7
+P 9200 1850
+F 0 "U1" H 8800 2450 50  0000 L CNN
+F 1 "NRF24L01-BRKOUT" H 9200 1250 50  0000 L CNN
+F 2 "NRF24L01-BKKOUT" H 9200 1850 50  0001 L CNN
+F 3 "" H 9200 1850 60  0000 C CNN
+	1    9200 1850
+	1    0    0    -1
+$EndComp
 $EndSCHEMATC
