File: documents/electronic design/beamer/_saved_beamer.sch (KiCad schematic (older format))
At the start: 28 parts, among them P1 CONN_01X20, P2 CONN_01X20, P3 CONN_01X02, P4 CONN_01X01, P5 CONN_01X01, T1 2N7002K, T10 2N7002K, T2 2N7002K, T3 2N7002K, T4 2N7002K, T5 2N7002K, T6 2N7002K, T7 2N7002K, T8 2N7002K, T9 2N7002K, U1 NRF24L01-BRKOUT, U2 74HC595D

Commit message: minor update in beamer pcb layout
Parts:
- C1: footprint (none) -> Capacitors_SMD:C_0402
- U1: symbol NRF24L01-BRKOUT -> NRF24L01-BRKOUT-RESCUE-beamer
Connections:
- net NRF_CE1: now also U1.3 (CE); no longer U1.4 (CSN)
- net NRF_CSN1: now also U1.4 (CSN); no longer U1.8 (IRQ)
- net NRF_IRQ1: now also U1.8 (IRQ); no longer U1.3 (CE)
Changed lines of the file:
@@
 EESchema Schematic File Version 2
+LIBS:beamer-rescue
 LIBS:power
 LIBS:device
@@
 F 0 "C1" H 8025 1700 50  0000 L CNN
 F 1 "C" H 8025 1500 50  0000 L CNN
-F 2 "" H 8038 1450 50  0001 C CNN
+F 2 "Capacitors_SMD:C_0402" H 8038 1450 50  0001 C CNN
 F 3 "" H 8000 1600 50  0000 C CNN
 	1    8000 1600
@@
 NoConn ~ 2800 5100
 $Comp
-L NRF24L01-BRKOUT U1
+L NRF24L01-BRKOUT-RESCUE-beamer U1
 U 1 1 576CC048
 P 8850 1800
