File: documents/electronic design/beamer/beamer.sch (KiCad schematic (older format))
At the start: 30 parts, among them P1 CONN_01X20, P2 CONN_01X20, P3 CONN_01X02, P4 CONN_01X01, P5 CONN_01X01, T1 2N7002K, T10 2N7002K, T2 2N7002K, T3 2N7002K, T4 2N7002K, T5 2N7002K, T6 2N7002K, T7 2N7002K, T8 2N7002K, T9 2N7002K, U1 NRF24L01-BRKOUT, U2 74HC595D

Commit message: save changes
Parts:
- removed P?: CONN_STM32F103_R_01X20, symbol CONN_STM32F103_R_01X20
- removed P?: CONN_STM32F103_L_01X20, symbol CONN_STM32F103_L_01X20
- removed U1: NRF24L01-BRKOUT, SE8R01:se8r01_smd, symbol NRF24L01-BRKOUT-RESCUE-beamer
- added P6, P8: CONN_01X08, Pin_Headers:Pin_Header_Straight_1x08, symbol CONN_01X08
- added P7, P9: CONN_01X04, Pin_Headers:Pin_Header_Straight_1x04, symbol CONN_01X04
- added U3: 74HC595D, 74HC595:SO16, symbol 74HC595D
- added U? (x2): NRF24L01-BRKOUT, NRF24L01-BKKOUT, symbol NRF24L01-BRKOUT
Connections:
- net +3V3: now also U?.1 (VCC)
- net GND: now also U?.2 (GND)
- net NRF_CE1: now also U?.3 (CE)
- net NRF_CSN1: now also U?.4 (CSN)
- net NRF_IRQ1: now also U?.8 (IRQ)
- net SPI1_MISO: now also U?.7 (MISO)
- net SPI1_MOSI: now also U?.6 (MOSI)
- net SPI1_SCK: now also U?.5 (SCK)
- new net: P8.1 (P1), U3.1 (Q1)
- new net: P6.2 (P2), U3.10 (~MR)
- new net: P6.3 (P3), U3.11 (SH_CP)
- new net: P6.4 (P4), U3.12 (ST_CP)
- new net: P6.5 (P5), U3.13 (~OE)
- new net: P6.6 (P6), U3.14 (DS)
- new net: P6.7 (P7), U3.15 (Q0)
- new net: P6.8 (P8), U3.16 (VCC)
- new net: P8.2 (P2), U3.2 (Q2)
- new net: P8.3 (P3), U3.3 (Q3)
- new net: P8.4 (P4), U3.4 (Q4)
- new net: P8.5 (P5), U3.5 (Q5)
- new net: P8.6 (P6), U3.6 (Q6)
- new net: P8.7 (P7), U3.7 (Q7)
- new net: P8.8 (P8), U3.8 (GND)
- new net: P6.1 (P1), U3.9 (Q7_2)
- new net: P9.1 (P1), U?.5 (SCK)
- new net: P9.2 (P2), U?.6 (MOSI)
- new net: P9.3 (P3), U?.7 (MISO)
- new net: P9.4 (P4), U?.8 (IRQ)
- new net: P7.1 (P1), U?.1 (VCC)
- new net: P7.2 (P2), U?.2 (GND)
- new net: P7.3 (P3), U?.3 (CE)
- new net: P7.4 (P4), U?.4 (CSN)
