File: documents/electronic design/ir_sensor/ir_sensor.sch (KiCad schematic (older format))
At the start: 11 parts, among them P1 Via, P2 Via, P3 Via, P4 Via, P5 Via, U1 TL1838, U2 STM32F103HEADER, U3 MPU6050_module, U4 SE8R01_module

Commit message: update pin mapping, regenerate for i2c2,spi2, number of tim input channels. WIP
Parts:
- removed C2: 100uf, Capacitors_SMD:C_1206_HandSoldering, symbol C
- removed P1, P2, P3, P4, P5: Via, footprints:Via, symbol Via
- removed U1: TL1838, footprints:TL1838_footprint, symbol TL1838
- added J1, J3, J4: Conn_01x12, Pin_Headers:Pin_Header_Straight_1x12_Pitch2.54mm, symbol Conn_01x12
- added J2: Conn_01x01, Pin_Headers:Pin_Header_Straight_1x01_Pitch2.54mm, symbol Conn_01x01
- U4: symbol SE8R01_module -> SE8R01_module-RESCUE-ir_sensor
Connections:
- net +3V3: now also J4.1 (Pin_1), J4.10 (Pin_10), J4.11 (Pin_11), J4.12 (Pin_12), J4.2 (Pin_2), J4.3 (Pin_3), J4.4 (Pin_4), J4.5 (Pin_5), J4.6 (Pin_6), J4.7 (Pin_7), J4.8 (Pin_8), J4.9 (Pin_9)
- net AD0: now also U2.32 (A4); no longer U2.35 (A1)
- net GND: now also J3.1 (Pin_1), J3.10 (Pin_10), J3.11 (Pin_11), J3.12 (Pin_12), J3.2 (Pin_2), J3.3 (Pin_3), J3.4 (Pin_4), J3.5 (Pin_5), J3.6 (Pin_6), J3.7 (Pin_7), J3.8 (Pin_8), J3.9 (Pin_9)
- net I2C_SCL: now also U2.26 (B10); no longer U2.16 (B8)
- net I2C_SDA: now also U2.25 (B11); no longer U2.17 (B9)
- net MPU5060_INT: now also U2.31 (A5); no longer U2.36 (A0)
- net SE8R01_CE: now also U2.6 (A9); no longer U2.7 (A10)
- net SE8R01_CSN: now also U2.5 (A8); no longer U2.8 (A11)
- net SE8R01_IRQ: now also U2.7 (A10); no longer U2.28 (B0)
- net SPI_MISO: now also U2.3 (B14); no longer U2.30 (A6)
- net SPI_MOSI: now also U2.4 (B15); no longer U2.29 (A7)
- net SPI_SCK: now also U2.2 (B13); no longer U2.31 (A5)
- net input_12: now reaches U2.10 (A15)
- net input_12: now also J1.1 (Pin_1)
- net input_11: now reaches U2.11 (B3)
- net input_11: now also J1.2 (Pin_2)
- net input_8: now reaches U2.15 (B7)
- net input_8: now also J1.4 (Pin_4)
- net input_6: now reaches U2.27 (B1)
- net input_6: now also J1.12 (Pin_12)
- net input_2: now reaches U2.33 (A3)
- net input_2: now also J1.8 (Pin_8)
- net input_1: now reaches U2.34 (A2)
- net input_1: now also J1.7 (Pin_7)
- net IR_RCV renamed input_7
- net input_7: now also J1.3 (Pin_3)
- new net LED_DBG: J2.1 (Pin_1), U2.36 (A0)
- new net input_10: J1.6 (Pin_6), U2.17 (B9)
- new net input_3: J1.9 (Pin_9), U2.30 (A6)
- new net input_4: J1.10 (Pin_10), U2.29 (A7)
- new net input_5: J1.11 (Pin_11), U2.28 (B0)
- new net input_9: J1.5 (Pin_5), U2.16 (B8)
- no-connect marks 25 -> 13
Other:
- note added: "* A8 OUT CSN \n * A9 OUT CE \n * A10 IN IRQ \n * A4 OUT MPU5060_AD0 \n * A5 IN MPU5060_INT \n * C13 OUT LED_ONBOARD \n * A0 OUT LED_DBG \n\nA15 tim2\nB3 tim2\nA2 tim2\nA3 tim2\nA6 tim3\nA7 tim3\nB0 tim3\nB1 tim3\nB6 tim4\nB7 tim4\nB8 tim4\nB9 tim4\n\nI2C:\nB10 SCL\nB11 SDA\n\nSPI:\nB13 SCK\nB14 MISO\nB15 MOSI\n\n"
- note removed: "I2C1:\nPB8 ------> I2C1_SCL\nPB9 ------> I2C1_SDA\n\n SPI1:\nMISO ------>A6\nMOSI ------>A7\nSCK ------>A5\n\n SE8R01:\nCSN ------> A11\nCE ------> A10\nIRQ ------> B0"
