File: documents/electronic design/ir_sensor/_saved_ir_sensor.sch (KiCad schematic (older format))
At the start: 11 parts, among them J2 Conn_01x01, U2 STM32F103HEADER, U3 MPU6050_module, U4 SE8R01_module

Commit message: adjust pcb design
Parts:
- J1, J3, J4, J5, J6, J7: renamed from J?; footprint (none) -> Pin_Headers:Pin_Header_Straight_1x06_Pitch2.54mm
Changed lines of the file:
@@
 $EndComp
 $Comp
-L Conn_01x06 J?
+L Conn_01x06 J3
 U 1 1 59FC2749
 P 1500 4200
-F 0 "J?" H 1500 4500 50  0000 C CNN
+F 0 "J3" H 1500 4500 50  0000 C CNN
 F 1 "Conn_01x06" H 1500 3800 50  0000 C CNN
-F 2 "" H 1500 4200 50  0001 C CNN
+F 2 "Pin_Headers:Pin_Header_Straight_1x06_Pitch2.54mm" H 1500 4200 50  0001 C CNN
 F 3 "" H 1500 4200 50  0001 C CNN
 	1    1500 4200
@@
 $EndComp
 $Comp
-L Conn_01x06 J?
+L Conn_01x06 J5
 U 1 1 59FC2827
 P 2300 4200
-F 0 "J?" H 2300 4500 50  0000 C CNN
+F 0 "J5" H 2300 4500 50  0000 C CNN
 F 1 "Conn_01x06" H 2300 3800 50  0000 C CNN
-F 2 "" H 2300 4200 50  0001 C CNN
+F 2 "Pin_Headers:Pin_Header_Straight_1x06_Pitch2.54mm" H 2300 4200 50  0001 C CNN
 F 3 "" H 2300 4200 50  0001 C CNN
 	1    2300 4200
@@
 $EndComp
 $Comp
-L Conn_01x06 J?
+L Conn_01x06 J7
 U 1 1 59FC2879
 P 3100 4200
-F 0 "J?" H 3100 4500 50  0000 C CNN
+F 0 "J7" H 3100 4500 50  0000 C CNN
 F 1 "Conn_01x06" H 3100 3800 50  0000 C CNN
-F 2 "" H 3100 4200 50  0001 C CNN
+F 2 "Pin_Headers:Pin_Header_Straight_1x06_Pitch2.54mm" H 3100 4200 50  0001 C CNN
 F 3 "" H 3100 4200 50  0001 C CNN
 	1    3100 4200
@@
 $EndComp
 $Comp
-L Conn_01x06 J?
+L Conn_01x06 J1
 U 1 1 59FC2A4E
 P 1500 3400
-F 0 "J?" H 1500 3700 50  0000 C CNN
+F 0 "J1" H 1500 3700 50  0000 C CNN
 F 1 "Conn_01x06" H 1500 3000 50  0000 C CNN
-F 2 "" H 1500 3400 50  0001 C CNN
+F 2 "Pin_Headers:Pin_Header_Straight_1x06_Pitch2.54mm" H 1500 3400 50  0001 C CNN
 F 3 "" H 1500 3400 50  0001 C CNN
 	1    1500 3400
@@
 $EndComp
 $Comp
-L Conn_01x06 J?
+L Conn_01x06 J4
 U 1 1 59FC2A54
 P 2300 3400
-F 0 "J?" H 2300 3700 50  0000 C CNN
+F 0 "J4" H 2300 3700 50  0000 C CNN
 F 1 "Conn_01x06" H 2300 3000 50  0000 C CNN
-F 2 "" H 2300 3400 50  0001 C CNN
+F 2 "Pin_Headers:Pin_Header_Straight_1x06_Pitch2.54mm" H 2300 3400 50  0001 C CNN
 F 3 "" H 2300 3400 50  0001 C CNN
 	1    2300 3400
@@
 $EndComp
 $Comp
-L Conn_01x06 J?
+L Conn_01x06 J6
 U 1 1 59FC2A5A
 P 3100 3400
-F 0 "J?" H 3100 3700 50  0000 C CNN
+F 0 "J6" H 3100 3700 50  0000 C CNN
 F 1 "Conn_01x06" H 3100 3000 50  0000 C CNN
-F 2 "" H 3100 3400 50  0001 C CNN
+F 2 "Pin_Headers:Pin_Header_Straight_1x06_Pitch2.54mm" H 3100 3400 50  0001 C CNN
 F 3 "" H 3100 3400 50  0001 C CNN
 	1    3100 3400
@@
 Connection ~ 1900 3300
 $Comp
-L GND #PWR?
+L GND #PWR012
 U 1 1 59FC2E26
 P 1900 4250
-F 0 "#PWR?" H 1900 4000 50  0001 C CNN
+F 0 "#PWR012" H 1900 4000 50  0001 C CNN
 F 1 "GND" H 1900 4100 50  0000 C CNN
 F 2 "" H 1900 4250 50  0000 C CNN
@@
 Connection ~ 2700 4100
 $Comp
-L +3V3 #PWR?
+L +3V3 #PWR013
 U 1 1 59FC2F1A
 P 2700 3450
-F 0 "#PWR?" H 2700 3300 50  0001 C CNN
+F 0 "#PWR013" H 2700 3300 50  0001 C CNN
 F 1 "+3V3" H 2700 3590 50  0000 C CNN
 F 2 "" H 2700 3450 50  0000 C CNN
@@
 $EndComp
 $Comp
-L +3V3 #PWR?
+L +3V3 #PWR014
 U 1 1 59FC2FFF
 P 2700 4250
-F 0 "#PWR?" H 2700 4100 50  0001 C CNN
+F 0 "#PWR014" H 2700 4100 50  0001 C CNN
 F 1 "+3V3" H 2700 4390 50  0000 C CNN
 F 2 "" H 2700 4250 50  0000 C CNN
